File: pcb/hb-bob/kicad-src/hb-bob-r1p0.kicad_pcb (KiCad board)
At the start: 2 copper layers, 30 x 30 mm, 67 parts, among them J1 PH_01x05, J2 PinHeader 1x02, J3 Terminal Block 2P, U1 CA-IS3720, U2 CA-IS3720, U3 74LVC2G14DW-7, U4 MAX22088

Commit message: wip: combined into one pcb
Parts:
- removed H1, H2, H3, H4: MountingHole, MountingHole:MountingHole_3.2mm_M3_DIN965
- removed J1: PH_01x05, Connector_PinHeader_2.54mm:PinHeader_1x05_P2.54mm_Vertical
- removed J2: PinHeader 1x02, Connector_PinHeader_2.54mm:PinHeader_1x02_P2.54mm_Vertical
- removed kibuzzard-65B62A1A (x2): G***, kibuzzard-65B62A1A
- removed kibuzzard-65B62B19 (x2): G***, kibuzzard-65B62B19
- removed kibuzzard-65B62B21 (x2): G***, kibuzzard-65B62B21
- removed the kibuzzard-65B6C60D at (187.1, 89.4)
- removed the kibuzzard-65B6C61A at (187.1, 85.5)
- removed kibuzzard-65B9E354: G***, kibuzzard-65B9E354
- removed kibuzzard-662F7DF1: G***, kibuzzard-662F7DF1
- removed kibuzzard-662F7DF9: G***, kibuzzard-662F7DF9
- removed kibuzzard-662F7E09: G***, kibuzzard-662F7E09
- removed kibuzzard-662F7E13: G***, kibuzzard-662F7E13
- added C12: 10uF, Capacitor_SMD:C_0603_1608Metric, F.Cu at (138.4, 107.2)
- added C13: 33nF, Capacitor_SMD:C_0402_1005Metric, F.Cu at (132.2, 104.2)
- added C14: 220nF, Capacitor_SMD:C_0402_1005Metric, F.Cu at (133.2, 107.5)
- added C15: 220nF, Capacitor_SMD:C_0402_1005Metric, F.Cu at (129.0, 107.5)
- added C16: 10uF, Capacitor_SMD:C_0603_1608Metric, F.Cu at (130.3, 107.5)
- added C17: 22uF, Capacitor_SMD:C_0603_1608Metric, F.Cu at (131.9, 107.5)
- added D10: ORANGE, LED_SMD:LED_0402_1005Metric, F.Cu at (127.9, 76.8)
- added D11: CUS10S30,H3F, Diode_SMD:D_SOD-523, F.Cu at (130.3, 105.1)
- added L1: 4.7uF, Inductor_SMD:L_0805_2012Metric, F.Cu at (129.9, 103.4)
- added R19: 5.1K, Resistor_SMD:R_0402_1005Metric, F.Cu at (139.4, 76.1)
- added R20: 5.1K, Resistor_SMD:R_0402_1005Metric, F.Cu at (138.2, 76.1)
- added R21: 2.2K, Resistor_SMD:R_0402_1005Metric, F.Cu at (143.1, 76.1)
- added R22: 2.2K, Resistor_SMD:R_0402_1005Metric, F.Cu at (141.9, 76.1)
- added R23: 470R, Resistor_SMD:R_0402_1005Metric, F.Cu at (127.9, 77.9)
- added R24: 49.9k, Resistor_SMD:R_0402_1005Metric, F.Cu at (135.5, 107.5)
- added R25: 15.8k, Resistor_SMD:R_0402_1005Metric, F.Cu at (134.4, 107.5)
- added TP1: UART_RXD, TestPoint:TestPoint_Pad_D1.0mm, F.Cu at (142.9, 93.5)
- added TP11: GND, TestPoint:TestPoint_Pad_D1.0mm, F.Cu at (131.7, 79.7)
- added TP12: 3V3, TestPoint:TestPoint_Pad_D1.0mm, F.Cu at (134.0, 79.8)
- added TP2: UART_TXD, TestPoint:TestPoint_Pad_D1.0mm, F.Cu at (145.3, 93.5)
- added TP3: RST, TestPoint:TestPoint_Pad_D1.0mm, F.Cu at (140.6, 93.5)
- added TP4: JDB_CTRL, TestPoint:TestPoint_Pad_D1.0mm, F.Cu at (138.2, 93.5)
- added TP8: I2C_SCL, TestPoint:TestPoint_Pad_D1.0mm, F.Cu at (134.1, 76.8)
- added TP9: I2C_SDA, TestPoint:TestPoint_Pad_D1.0mm, F.Cu at (131.8, 76.8)
- added U5: ESP32-C3-MINI-1, lib:ESP32-C3-MINI-1, F.Cu at (144.2, 84.5)
- added U6: AOZ1280CI, Package_TO_SOT_SMD:SOT-23-6, F.Cu at (134.4, 104.4)
- added kibuzzard-68B31F11: G***, kibuzzard-68B31F11, F.Cu at (121.4, 80.0)
- added kibuzzard-68B31F54: G***, kibuzzard-68B31F54, F.Cu at (128.0, 75.7)
- added kibuzzard-68B31FE4: G***, kibuzzard-68B31FE4, F.Cu at (119.1, 79.0)
- added kibuzzard-68B32675: G***, kibuzzard-68B32675, F.Cu at (131.5, 78.3)
- added kibuzzard-68B326CE: G***, kibuzzard-68B326CE, F.Cu at (142.9, 92.0)
- added kibuzzard-68B326E4: G***, kibuzzard-68B326E4, F.Cu at (145.2, 92.0)
- added kibuzzard-68B326FE: G***, kibuzzard-68B326FE, F.Cu at (140.6, 92.0)
- added kibuzzard-68B3271E: G***, kibuzzard-68B3271E, F.Cu at (138.2, 92.0)
- added kibuzzard-68B32731: G***, kibuzzard-68B32731, F.Cu at (131.8, 75.2)
- added kibuzzard-68B3273B: G***, kibuzzard-68B3273B, F.Cu at (134.2, 75.3)
- added kibuzzard-68B32786: G***, kibuzzard-68B32786, F.Cu at (134.0, 78.3)
- C4: footprint Capacitor_SMD:CP_Elec_6.3x7.7 -> Capacitor_Tantalum_SMD:CP_EIA-7360-38_Kemet-E_Pad2.25x4.25mm_HandSolder
- J3: value Terminal Block 2P -> Conn_01x02_Pin; footprint Connector_Phoenix_MC:PhoenixContact_MC_1,5_2-G-3.81_1x02_P3.81mm_Horizontal -> Connector_PinHeader_2.54mm:PinHeader_1x02_P2.54mm_Horizontal
- moved kibuzzard-65B6C60D 77.5 mm to (112.9, 101.1), turned to -90 degrees
- moved kibuzzard-65B6C61A 73.4 mm to (119.2, 101.3), turned to -90 degrees
- moved J3 67.6 mm to (117.3, 101.0), turned to -90 degrees
- moved D6 63.8 mm to (118.3, 93.0), turned to 180 degrees
- moved R14 63.6 mm to (114.4, 92.5), turned to -90 degrees
- moved D4 62.2 mm to (115.2, 96.8), turned to -90 degrees
- moved D9 61.6 mm to (118.7, 96.8), turned to -90 degrees
- moved R12 58.8 mm to (115.6, 77.7), turned to 180 degrees
- moved U3 57.1 mm to (117.6, 83.2)
- moved R11 55.8 mm to (123.3, 99.9), turned to 180 degrees
- moved C10 55.4 mm to (120.2, 107.7), turned to 90 degrees
- moved C11 55.1 mm to (120.2, 103.8), turned to 90 degrees
- moved D5 54.7 mm to (115.6, 76.7)
- moved kibuzzard-65B629C5 54.7 mm to (115.7, 75.6)
- moved C9 54.4 mm to (126.6, 100.8)
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Connections:
- C1 pad 2: /IOGND -> GND
- D1 pad 1: /IOGND -> GND
- J3 pad 1: /H+ -> /H-
- J3 pad 2: /H- -> /H+
- U1 pad 4: /IOGND -> GND
- U2 pad 5: /IOGND -> GND
Routing:
- net VCC: track 41.7 -> 0.00 mm, vias 5 -> 0
- net GND: track 29.8 -> 0.00 mm, vias 24 -> 0
- net /IOGND: track 28.6 -> 0.00 mm, vias 3 -> 0
- net /_DOUT: track 24.2 -> 0.00 mm, vias 2 -> 0
- net /IOVDD: track 21.3 -> 0.00 mm
- net /H-: track 20.3 -> 0.00 mm
- net /RST: track 16.7 -> 0.00 mm, vias 1 -> 0
- net Net-(D8-A1): track 16.3 -> 0.00 mm, vias 2 -> 0
- net Net-(D6-A1): track 14.7 -> 0.00 mm, vias 2 -> 0
- net /_DIN: track 13.6 -> 0.00 mm, vias 2 -> 0
- net /VRAW: track 4.42 -> 17.4 mm
- net Net-(D7-A1): track 12.6 -> 0.00 mm, vias 2 -> 0
- net /DIN: track 12.4 -> 0.00 mm, vias 1 -> 0
- net /H+: track 11.5 -> 0.00 mm
- net Net-(U4-HP): track 11.5 -> 0.00 mm, vias 2 -> 0
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Other:
- board size 30 x 30 mm -> 35 x 35 mm
- board text removed: "DI"
- board text removed: "DO"
- board text removed: "GND"
- board text removed: "RS"
- board text removed: "VDD"
