File: pcb/hb-bob/kicad-src/hb-bob-r1p0.kicad_sch (KiCad schematic)
At the start: 49 parts, among them J1 PH_01x05, J2 PinHeader 1x02, J3 Terminal Block 2P, U1 CA-IS3720, U2 CA-IS3720, U3 74LVC2G14DW-7, U4 MAX22088

Commit message: wip: combined into one pcb
Parts:
- removed H1, H2, H3, H4: MountingHole, MountingHole:MountingHole_3.2mm_M3_DIN965, symbol Mechanical:MountingHole
- removed J1: PH_01x05, Connector_PinHeader_2.54mm:PinHeader_1x05_P2.54mm_Vertical, symbol Connector:Conn_01x05_Male
- removed J2: PinHeader 1x02, Connector_PinHeader_2.54mm:PinHeader_1x02_P2.54mm_Vertical, symbol Connector:Conn_01x02_Male
- removed J3: Terminal Block 2P, Connector_Phoenix_MC:PhoenixContact_MC_1,5_2-G-3.81_1x02_P3.81mm_Horizontal, symbol Connector:Conn_01x02_Female
- added C12, C16: 10uF, Capacitor_SMD:C_0603_1608Metric, symbol Device:C
- added C13: 33nF, Capacitor_SMD:C_0402_1005Metric, symbol Device:C
- added C14, C15: 220nF, Capacitor_SMD:C_0402_1005Metric, symbol Device:C
- added C17: 22uF, Capacitor_SMD:C_0603_1608Metric, symbol Device:C
- added D10: ORANGE, LED_SMD:LED_0402_1005Metric, symbol Device:LED_Filled
- added D11: CUS10S30,H3F, Diode_SMD:D_SOD-523, symbol Device:D_Schottky_Filled
- added J3: Conn_01x02_Pin, Connector_PinHeader_2.54mm:PinHeader_1x02_P2.54mm_Horizontal, symbol Connector:Conn_01x02_Pin
- added L1: 4.7uF, Inductor_SMD:L_0805_2012Metric, symbol Device:L
- added R19, R20: 5.1K, Resistor_SMD:R_0402_1005Metric, symbol Device:R
- added R21, R22: 2.2K, Resistor_SMD:R_0402_1005Metric, symbol Device:R
- added R23: 470R, Resistor_SMD:R_0402_1005Metric, symbol Device:R
- added R24: 49.9k, Resistor_SMD:R_0402_1005Metric, symbol Device:R
- added R25: 15.8k, Resistor_SMD:R_0402_1005Metric, symbol Device:R
- added TP1: UART_RXD, TestPoint:TestPoint_Pad_D1.0mm, symbol Connector:TestPoint_Alt
- added TP11: GND, TestPoint:TestPoint_Pad_D1.0mm, symbol Connector:TestPoint_Alt
- added TP12: 3V3, TestPoint:TestPoint_Pad_D1.0mm, symbol Connector:TestPoint_Alt
- added TP2: UART_TXD, TestPoint:TestPoint_Pad_D1.0mm, symbol Connector:TestPoint_Alt
- added TP3: RST, TestPoint:TestPoint_Pad_D1.0mm, symbol Connector:TestPoint_Alt
- added TP4: JDB_CTRL, TestPoint:TestPoint_Pad_D1.0mm, symbol Connector:TestPoint_Alt
- added TP8: I2C_SCL, TestPoint:TestPoint_Pad_D1.0mm, symbol Connector:TestPoint_Alt
- added TP9: I2C_SDA, TestPoint:TestPoint_Pad_D1.0mm, symbol Connector:TestPoint_Alt
- added U5: ESP32-C3-MINI-1, lib:ESP32-C3-MINI-1, symbol lib:ESP32-C3-MINI-1
- added U6: AOZ1280CI, Package_TO_SOT_SMD:SOT-23-6, symbol Regulator_Switching:AOZ1280CI
- C4: footprint Capacitor_SMD:CP_Elec_6.3x7.7 -> Capacitor_Tantalum_SMD:CP_EIA-7360-38_Kemet-E_Pad2.25x4.25mm_HandSolder
Connections:
- net IOGND is gone; now on net GND: C1.2, D1.1 (K), U1.4 (GND1), U2.5 (GND2)
- net DIN: now also R22.2, TP9.1, U5.6 (GPIO3/ADC1_CH3)
- net DOUT: now also R21.2, TP8.1, U5.5 (GPIO2/ADC1_CH2)
- net GND: now also C12.2, C14.2, C15.2, C16.2, C17.2, D10.1 (K), D11.2 (A), R25.2, TP11.1, U5.1 (GND), U5.11 (GND), U5.14 (GND), U5.2 (GND), U5.36 (GND), U5.37 (GND), U5.38 (GND), U5.39 (GND), U5.40 (GND), U5.41 (GND), U5.42 (GND), U5.43 (GND), U5.44 (GND), U5.45 (GND), U5.46 (GND), U5.47 (GND), U5.48 (GND), U5.49 (GND), U5.50 (GND), U5.51 (GND), U5.52 (GND), U5.53 (GND), U6.2 (GND)
- net H+: now also J3.2 (Pin_2)
- net H-: now also J3.1 (Pin_1)
- net RST: now also U5.16 (GPIO10)
- net VRAW: now also C12.1, U6.4 (EN), U6.5 (VIN)
- new net: TP4.1, U5.23 (GPIO9)
- new net: R24.2, R25.1, U6.3 (FB)
- new net: R19.2, TP3.1, U5.8 (EN/CHIP_PU)
- new net: C13.1, D11.1 (K), L1.1, U6.6 (LX)
- new net: C13.2, U6.1 (BST)
- new net: D10.2 (A), R23.1
- new net: R23.2, U5.18 (GPIO4/ADC1_CH4)
- new net: TP1.1, U5.30 (GPIO20/U0RXD)
- new net: TP2.1, U5.31 (GPIO21/U0TXD)
- new net: R20.2, U5.22 (GPIO8)
- new net +3V3: C14.1, C15.1, C16.1, C17.1, L1.2, R19.1, R20.1, R21.1, R22.1, R24.1, TP12.1, U5.3 (3V3)
- no-connect marks 1 -> 8
